File: adat_output.sch (KiCad schematic (older format))
At the start: 9 parts, among them U301 V1401, U302 74LVC1G04, U303 74LVC1G04

Commit message: Remove dependency on digikey libraries.
Parts:
- U302, U303: symbol 74xGxx:74LVC1G04 -> gradator:74LVC1GU04
Changed lines of the file:
@@
 in1
 $Comp
-L 74xGxx:74LVC1G04 U302
+L gradator:74LVC1GU04 U302
 U 1 1 605B6B6C
 P 7650 2650
@@
 	7950 3400 8750 3400
 $Comp
-L 74xGxx:74LVC1G04 U303
+L gradator:74LVC1GU04 U303
 U 1 1 6031D59B
 P 7850 4600
