File: input.sch (KiCad schematic (older format))
At the start: 20 parts, among them U1 74AHC1G04

Commit message: Remove dependency on digikey libraries.
Parts:
- DIR1: footprint digikey-footprints:TSSOP-28_W4.40mm -> Package_SO:TSSOP-28_4.4x9.7mm_P0.65mm
- SRC11: footprint digikey-footprints:SSOP-28_W5.30mm -> Package_SO:SSOP-28_5.3x10.2mm_P0.65mm
Changed lines of the file:
@@
 F 0 "SRC11" H 9300 3850 50  0000 C CNN
 F 1 "SRC4190" H 9300 3750 50  0000 C CNN
-F 2 "digikey-footprints:SSOP-28_W5.30mm" H 8950 4050 50  0001 C CNN
+F 2 "Package_SO:SSOP-28_5.3x10.2mm_P0.65mm" H 8950 4050 50  0001 C CNN
 F 3 "" H 8900 3000 50  0001 C CNN
 	1    8900 3100
@@
 F 0 "DIR1" H 5550 2950 50  0000 C CNN
 F 1 "DIR9001" H 5550 2850 50  0000 C CNN
-F 2 "digikey-footprints:TSSOP-28_W4.40mm" H 5250 2550 50  0001 C CNN
+F 2 "Package_SO:TSSOP-28_4.4x9.7mm_P0.65mm" H 5250 2550 50  0001 C CNN
 F 3 "" H 5250 2550 50  0001 C CNN
 	1    5250 2550
